File: Interface/Hardware/interfacer/debugging_LEDs.sch (KiCad schematic (older format))
At the start: 17 parts, among them U1 ULN2003A

Commit message: antenna power touch-up & green LED resistor value change
Parts:
- R5, R7, R9: value 1k5 -> 10k
Changed lines of the file:
@@
 P 6200 3350
 F 0 "R5" V 6280 3350 50  0000 C CNN
-F 1 "1k5" V 6200 3350 50  0000 C CNN
+F 1 "10k" V 6200 3350 50  0000 C CNN
 F 2 "auxiliary:0805_2012" V 6130 3350 50  0001 C CNN
 F 3 "" H 6200 3350 50  0001 C CNN
@@
 P 7000 3350
 F 0 "R7" V 7080 3350 50  0000 C CNN
-F 1 "1k5" V 7000 3350 50  0000 C CNN
+F 1 "10k" V 7000 3350 50  0000 C CNN
 F 2 "auxiliary:0805_2012" V 6930 3350 50  0001 C CNN
 F 3 "" H 7000 3350 50  0001 C CNN
@@
 P 7800 3350
 F 0 "R9" V 7880 3350 50  0000 C CNN
-F 1 "1k5" V 7800 3350 50  0000 C CNN
+F 1 "10k" V 7800 3350 50  0000 C CNN
 F 2 "auxiliary:0805_2012" V 7730 3350 50  0001 C CNN
 F 3 "" H 7800 3350 50  0001 C CNN
