File: Interface/Hardware/interfacer/main_connector.sch (KiCad schematic (older format))
At the start: 6 parts, among them J19 left top conn, J20 right top conn, J8 left bottom conn, J9 right bottom conn

Commit message: GPS module, PPS feedback 50 ohm drive, molex connectors
Other:
- note added: "this is useless\na crossover cable is needed instead"
- note removed: "this is useless\na cross cable is needed instead"
Changed lines of the file:
@@
 	4000 4050 4650 4050
 Wire Wire Line
-	7250 3850 7900 3850
+	7250 3850 8000 3850
 Wire Wire Line
-	7900 3850 8000 3850
-Wire Wire Line
-	7250 3950 7850 3950
-Wire Wire Line
-	7850 3950 8000 3950
+	7250 3950 8000 3950
 Wire Wire Line
 	7250 4450 8000 4450
@@
 Connection ~ 8550 3200
 Wire Wire Line
-	8550 3150 8550 3200
-Wire Wire Line
-	8550 3200 8550 3250
+	8550 3150 8550 3250
 Wire Wire Line
 	2050 1250 1900 1250
@@
 Connection ~ 7900 3850
 Text Notes 7900 4200 0    60   ~ 0
-this is useless\na cross cable is needed instead
+this is useless\na crossover cable is needed instead
 $EndSCHEMATC
